File: Polytuna KiCad/Polytuna.sch (KiCad schematic (older format))
At the start: 43 parts, among them IC1 AP7313-33SAG-7, J1 Barrel_Jack, J2 Conn_01x02, J3 Conn_01x02, J4 Conn_01x04, SW1 SW_Push, SW2 SW_Push, SW3 SW_Push, SW4 SW_DPDT_x2, U1 LM358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

Commit message: footprint-component relation finished
Parts:
- BOARD1: footprint (none) -> def-footprints:Board_Teensy_3_1
- BT1, J2, J3: footprint (none) -> Pin_Headers:Pin_Header_Straight_1x02_Pitch2.54mm
- D1, D2, D3: footprint (none) -> LEDs:LED_D3.0mm
- IC1: footprint (none) -> TO_SOT_Packages_SMD:SOT-23
- Input1, Output1: footprint (none) -> def-footprints:CONN_Jack_Female_6.35mm_THD
- J1: footprint (none) -> Connectors:Barrel_Jack_CUI_PJ-102AH
- J4: footprint (none) -> Pin_Headers:Pin_Header_Straight_1x04_Pitch2.54mm
- JMP1: footprint (none) -> def-footprints:Miscellaneous_Solder_Jumper
- RV1, RV2, RV3: footprint (none) -> Potentiometers:Potentiometer_Alps_RK09K_Horizontal
- SW1, SW2, SW3: footprint (none) -> Buttons_Switches_THT:SW_PUSH_6mm_h5mm
- SW4: footprint (none) -> def-footprints:Switches_Stomp_Switch_3PDT
- U3: footprint (none) -> TO_SOT_Packages_THT:TO-220-3_Horizontal
Changed lines of the file:
@@
 F 0 "Input1" H 825 1825 50  0000 C CNN
 F 1 "Audio-Jack-2" H 825 1575 50  0000 C CNN
-F 2 "" H 1100 1750 50  0001 C CNN
+F 2 "def-footprints:CONN_Jack_Female_6.35mm_THD" H 1100 1750 50  0001 C CNN
 F 3 "" H 1100 1750 50  0001 C CNN
 	1    850  1750
@@
 F 0 "SW4" H 5650 4170 50  0000 C CNN
 F 1 "SW_DPDT_x2" H 5650 3800 50  0000 C CNN
-F 2 "" H 5650 4000 50  0001 C CNN
+F 2 "def-footprints:Switches_Stomp_Switch_3PDT" H 5650 4000 50  0001 C CNN
 F 3 "" H 5650 4000 50  0001 C CNN
 	2    5650 4000
@@
 F 0 "SW4" H 1650 1920 50  0000 C CNN
 F 1 "SW_DPDT_x2" H 1650 1550 50  0000 C CNN
-F 2 "" H 1650 1750 50  0001 C CNN
+F 2 "def-footprints:Switches_Stomp_Switch_3PDT" H 1650 1750 50  0001 C CNN
 F 3 "" H 1650 1750 50  0001 C CNN
 	1    1650 1750
@@
 F 0 "Output1" H 775 1175 50  0000 C CNN
 F 1 "Audio-Jack-2" H 775 925 50  0000 C CNN
-F 2 "" H 1050 1100 50  0001 C CNN
+F 2 "def-footprints:CONN_Jack_Female_6.35mm_THD" H 1050 1100 50  0001 C CNN
 F 3 "" H 1050 1100 50  0001 C CNN
 	1    800  1100
@@
 F 0 "BOARD1" H 4650 5000 60  0000 C CNN
 F 1 "BOARD_TEENSY_3.1" H 3250 5000 60  0000 C CNN
-F 2 "" H 3900 4850 60  0001 C CNN
+F 2 "def-footprints:Board_Teensy_3_1" H 3900 4850 60  0001 C CNN
 F 3 "" H 3900 4850 60  0000 C CNN
 	1    3900 5950
@@
 F 0 "JMP1" H 2050 895 60  0000 C CNN
 F 1 "2Jumper" H 2050 985 60  0001 C CNN
-F 2 "" H 3205 870 60  0001 C CNN
+F 2 "def-footprints:Miscellaneous_Solder_Jumper" H 3205 870 60  0001 C CNN
 F 3 "" H 3205 870 60  0000 C CNN
 	1    2050 800
@@
 F 0 "SW1" H 1900 4450 50  0000 L CNN
 F 1 "SW_Push" H 1850 4290 50  0000 C CNN
-F 2 "" H 1850 4550 50  0001 C CNN
+F 2 "Buttons_Switches_THT:SW_PUSH_6mm_h5mm" H 1850 4550 50  0001 C CNN
 F 3 "" H 1850 4550 50  0001 C CNN
 	1    1850 4350
@@
 F 0 "SW2" H 1850 4700 50  0000 L CNN
 F 1 "SW_Push" H 1800 4540 50  0000 C CNN
-F 2 "" H 1800 4800 50  0001 C CNN
+F 2 "Buttons_Switches_THT:SW_PUSH_6mm_h5mm" H 1800 4800 50  0001 C CNN
 F 3 "" H 1800 4800 50  0001 C CNN
 	1    1800 4600
@@
 F 0 "SW3" H 1850 4950 50  0000 L CNN
 F 1 "SW_Push" H 1800 4790 50  0000 C CNN
-F 2 "" H 1800 5050 50  0001 C CNN
+F 2 "Buttons_Switches_THT:SW_PUSH_6mm_h5mm" H 1800 5050 50  0001 C CNN
 F 3 "" H 1800 5050 50  0001 C CNN
 	1    1800 4850
@@
 F 0 "D1" H 1050 5550 50  0000 C CNN
 F 1 "LED" H 1050 5350 50  0000 C CNN
-F 2 "" H 1050 5450 50  0001 C CNN
+F 2 "LEDs:LED_D3.0mm" H 1050 5450 50  0001 C CNN
 F 3 "" H 1050 5450 50  0001 C CNN
 	1    1050 5450
@@
 F 0 "D2" H 1050 5800 50  0000 C CNN
 F 1 "LED" H 1050 5600 50  0000 C CNN
-F 2 "" H 1050 5700 50  0001 C CNN
+F 2 "LEDs:LED_D3.0mm" H 1050 5700 50  0001 C CNN
 F 3 "" H 1050 5700 50  0001 C CNN
 	1    1050 5700
@@
 F 0 "D3" H 1050 6050 50  0000 C CNN
 F 1 "LED" H 1050 5850 50  0000 C CNN
-F 2 "" H 1050 5950 50  0001 C CNN
+F 2 "LEDs:LED_D3.0mm" H 1050 5950 50  0001 C CNN
 F 3 "" H 1050 5950 50  0001 C CNN
 	1    1050 5950
@@
 F 0 "IC1" H 9200 1400 50  0000 L CNN
 F 1 "AP7313-33SAG-7" H 9200 1300 50  0000 L CNN
-F 2 "" H 9200 1200 50  0001 L CNN
+F 2 "TO_SOT_Packages_SMD:SOT-23" H 9200 1200 50  0001 L CNN
 F 3 "https://componentsearchengine.com/Datasheets/1/AP7313-33SAG-7.pdf" H 9200 1100 50  0001 L CNN
 F 4 "Diodes Inc AP7313-33SAG-7, Single Linear Voltage Regulator, 150mA 3.3 V, 2%, 3-Pin SOT-23" H 9200 1000 50  0001 L CNN "Description"
@@
 F 0 "RV1" V 6125 6050 50  0000 C CNN
 F 1 "POT_TRIM" V 6200 6050 50  0000 C CNN
-F 2 "" H 6300 6050 50  0001 C CNN
+F 2 "Potentiometers:Potentiometer_Alps_RK09K_Horizontal" H 6300 6050 50  0001 C CNN
 F 3 "" H 6300 6050 50  0001 C CNN
 	1    6300 6050
@@
 F 0 "RV3" V 6125 7200 50  0000 C CNN
 F 1 "POT_TRIM" V 6200 7200 50  0000 C CNN
-F 2 "" H 6300 7200 50  0001 C CNN
+F 2 "Potentiometers:Potentiometer_Alps_RK09K_Horizontal" H 6300 7200 50  0001 C CNN
 F 3 "" H 6300 7200 50  0001 C CNN
 	1    6300 7200
@@
 F 0 "RV2" V 6125 6650 50  0000 C CNN
 F 1 "POT_TRIM" V 6200 6650 50  0000 C CNN
-F 2 "" H 6300 6650 50  0001 C CNN
+F 2 "Potentiometers:Potentiometer_Alps_RK09K_Horizontal" H 6300 6650 50  0001 C CNN
 F 3 "" H 6300 6650 50  0001 C CNN
 	1    6300 6650
@@
 F 0 "J1" H 6650 4310 50  0000 C CNN
 F 1 "Barrel_Jack" H 6650 3925 50  0000 C CNN
-F 2 "" H 6700 4060 50  0001 C CNN
+F 2 "Connectors:Barrel_Jack_CUI_PJ-102AH" H 6700 4060 50  0001 C CNN
 F 3 "" H 6700 4060 50  0001 C CNN
 	1    6650 4100
@@
 F 0 "BT1" H 6000 4400 50  0000 L CNN
 F 1 "Battery" H 6000 4300 50  0000 L CNN
-F 2 "" V 5900 4360 50  0001 C CNN
+F 2 "Pin_Headers:Pin_Header_Straight_1x02_Pitch2.54mm" V 5900 4360 50  0001 C CNN
 F 3 "" V 5900 4360 50  0001 C CNN
 	1    5900 4300
@@
 F 0 "U3" H 4600 4025 50  0000 C CNN
 F 1 "L7805" H 4750 4025 50  0000 L CNN
-F 2 "" H 4775 3750 50  0001 L CIN
+F 2 "TO_SOT_Packages_THT:TO-220-3_Horizontal" H 4775 3750 50  0001 L CIN
 F 3 "" H 4750 3850 50  0001 C CNN
 	1    4750 3900
@@
 F 0 "J3" H 1350 3200 50  0000 C CNN
 F 1 "Conn_01x02" H 1350 2900 50  0000 C CNN
-F 2 "" H 1350 3100 50  0001 C CNN
+F 2 "Pin_Headers:Pin_Header_Straight_1x02_Pitch2.54mm" H 1350 3100 50  0001 C CNN
 F 3 "" H 1350 3100 50  0001 C CNN
 	1    1350 3100
@@
 F 0 "J2" H 1350 3700 50  0000 C CNN
 F 1 "Conn_01x02" H 1350 3400 50  0000 C CNN
-F 2 "" H 1350 3600 50  0001 C CNN
+F 2 "Pin_Headers:Pin_Header_Straight_1x02_Pitch2.54mm" H 1350 3600 50  0001 C CNN
 F 3 "" H 1350 3600 50  0001 C CNN
 	1    1350 3600
@@
 F 0 "J4" H 9500 6200 50  0000 C CNN
 F 1 "Conn_01x04" H 9500 5700 50  0000 C CNN
-F 2 "" H 9500 6000 50  0001 C CNN
+F 2 "Pin_Headers:Pin_Header_Straight_1x04_Pitch2.54mm" H 9500 6000 50  0001 C CNN
 F 3 "" H 9500 6000 50  0001 C CNN
 	1    9500 6000

Commit message: Progress in routing
Connections:
- net at BOARD1.10 (D8/TX3/DIN): now also R1.1
- net at BOARD1.2 (D0/RX1): no longer SW1.2
- net at BOARD1.3 (D1/TX1): no longer SW2.2
- net at BOARD1.4 (D2/CS): no longer SW3.2
- net at BOARD1.5 (D3/CAN_TX/PWM): now also SW1.2; no longer R3.1
- net at BOARD1.6 (D4/CAN_RX/PWM): now also SW2.2; no longer R2.1
- net at BOARD1.7 (D5/TX1/PWM): now also SW3.2; no longer R1.1
- net at BOARD1.8 (D6/CS/PWM): now also R3.1
- net at BOARD1.9 (D7/RX3/DOUT): now also R2.1
Changed lines of the file:
@@
 NoConn ~ 5100 5850
 NoConn ~ 5100 5950
-NoConn ~ 2700 6050
-NoConn ~ 2700 6150
-NoConn ~ 2700 6250
 NoConn ~ 2700 6450
 NoConn ~ 2700 6650
@@
 Connection ~ 2050 1100
 Wire Wire Line
-	2700 5450 2650 5450
-Wire Wire Line
-	2650 5450 2650 4350
-Wire Wire Line
 	2650 4350 2050 4350
 Wire Wire Line
-	2700 5550 2600 5550
-Wire Wire Line
-	2600 5550 2600 4600
+	2600 4600 2600 5850
 Wire Wire Line
 	2600 4600 2000 4600
 Wire Wire Line
-	2700 5650 2550 5650
-Wire Wire Line
-	2550 5650 2550 4850
+	2550 4850 2550 5950
 Wire Wire Line
 	2550 4850 2000 4850
 Wire Wire Line
-	2700 5750 2300 5750
-Wire Wire Line
-	2300 5750 2300 5450
+	2300 5450 2300 6050
 Wire Wire Line
 	1550 5450 1200 5450
 Wire Wire Line
-	2700 5850 2250 5850
-Wire Wire Line
-	2250 5850 2250 5700
+	2250 5700 2250 6150
 Wire Wire Line
 	1500 5700 1200 5700
-Wire Wire Line
-	1750 5950 2700 5950
 Wire Wire Line
 	1450 5950 1200 5950
@@
 Text Notes 8300 1750 0    60   ~ 0
 Maybe 1uF ??
+Wire Wire Line
+	1750 5950 2150 5950
+Wire Wire Line
+	2150 5950 2150 6250
+Wire Wire Line
+	2150 6250 2700 6250
+Wire Wire Line
+	2250 6150 2700 6150
+Wire Wire Line
+	2300 6050 2700 6050
+Wire Wire Line
+	2650 4350 2650 5750
+Wire Wire Line
+	2650 5750 2700 5750
+Wire Wire Line
+	2600 5850 2700 5850
+Wire Wire Line
+	2550 5950 2700 5950
+NoConn ~ 2700 5450
+NoConn ~ 2700 5550
+NoConn ~ 2700 5650
 $EndSCHEMATC

Commit message: Moar routing
Connections:
- net GND: now also U2.33 (GND)
- no-connect marks 18 -> 17
Changed lines of the file:
@@
 NoConn ~ 10050 3850
 NoConn ~ 10050 3700
-NoConn ~ 9750 4400
 NoConn ~ 10050 3500
 NoConn ~ 10050 3400
@@
 NoConn ~ 2700 5550
 NoConn ~ 2700 5650
+$Comp
+L GND #PWR?
+U 1 1 5AABFC35
+P 9750 4400
+F 0 "#PWR?" H 9750 4150 50  0001 C CNN
+F 1 "GND" H 9750 4250 50  0000 C CNN
+F 2 "" H 9750 4400 50  0001 C CNN
+F 3 "" H 9750 4400 50  0001 C CNN
+	1    9750 4400
+	1    0    0    -1
+$EndComp
 $EndSCHEMATC
